File: Digital_Clock_6_Digits.kicad_sch (KiCad schematic)
At the start: 0 parts

Commit message: Add backup files and create project settings for Digital Clock 6 Digits
- Added a backup zip file containing project files and settings.
- Created a new KiCad project settings file (Digital_Clock_6_Digits.kicad_prl) with configuration for board visibility, selection filters, and net inspector panel settings.
Other:
- added sheet 7Seg_6Digits (7Seg_6Digits.kicad_sch)
Changed lines of the file:
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@@
 	(generator_version "9.0")
 	(paper "A4")
+	(sheet
+		(at 87.63 99.06)
+		(size 58.42 20.955)
+		(exclude_from_sim no)
+		(in_bom yes)
+		(on_board yes)
+		(dnp no)
+		(fields_autoplaced yes)
+		(stroke
+			(width 0.1524)
+			(type solid)
+		)
+		(fill
+			(color 0 0 0 0.0000)
+		)
+		(property "Sheetname" "7Seg_6Digits"
+			(at 87.63 98.3484 0)
+			(effects
+				(font
+					(size 1.27 1.27)
+				)
+				(justify left bottom)
+			)
+		)
+		(property "Sheetfile" "7Seg_6Digits.kicad_sch"
+			(at 87.63 120.5996 0)
+			(effects
+				(font
+					(size 1.27 1.27)
+				)
+				(justify left top)
+			)
+		)
+		(instances
+			(project "Digital_Clock_6_Digits"
+				(path "/79d96a8f-9c80-4f83-a25e-7a8fff40baf7"
+					(page "2")
+				)
+			)
+		)
+	)
 	(sheet_instances
 		(path "/"
