File: Counter.kicad_sch (KiCad schematic)
At the start: 0 parts

Commit message: Add 74LS192 counter and project links
Add a 74LS192 symbol definition and instance to Counter.kicad_sch (includes pins, properties and a U1 instance). Update Digital_Clock_6_Digits.kicad_pro to register Controller, Seven_Segment_View and Counter modules. Update Seven_Segment_View.kicad_sch by replacing many concrete reference names with placeholders (R?, U?, #PWR?) and adding project/path metadata for those symbols so they link back to the Digital_Clock_6_Digits project. These changes integrate the new counter symbol into the project and prepare hierarchical symbol/project linking.
Parts:
- added U1: 74LS192, symbol 74xx:74LS192
Changed lines of the file:
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@@
 	(generator_version "9.0")
 	(paper "A4")
+	(wire
+		(pts
+			(xy 72.39 26.67) (xy 72.39 53.34)
+		)
+		(stroke
+			(width 0)
+			(type default)
+		)
+	)
+	(wire
+		(pts
+			(xy 60.96 50.8) (xy 69.85 50.8)
+		)
+		(stroke
+			(width 0)
+			(type default)
+		)
+	)
+	(wire
+		(pts
+			(xy 60.96 48.26) (xy 67.31 48.26)
+		)
+		(stroke
+			(width 0)
+			(type default)
+		)
+	)
+	(wire
+		(pts
+			(xy 60.96 53.34) (xy 72.39 53.34)
+		)
+		(stroke
+			(width 0)
+			(type default)
+		)
+	)
+	(wire
+		(pts
+			(xy 69.85 26.67) (xy 69.85 50.8)
+		)
+		(stroke
+			(width 0)
+			(type default)
+		)
+	)
+	(wire
+		(pts
+			(xy 67.31 26.67) (xy 67.31 48.26)
+		)
+		(stroke
+			(width 0)
+			(type default)
+		)
+	)
+	(wire
+		(pts
+			(xy 60.96 45.72) (xy 64.77 45.72)
+		)
+		(stroke
+			(width 0)
+			(type default)
+		)
+	)
+	(wire
+		(pts
+			(xy 64.77 26.67) (xy 64.77 45.72)
+		)
+		(stroke
+			(width 0)
+			(type default)
+		)
+	)
+	(symbol
+		(lib_id "74xx:74LS192")
+		(at 48.26 55.88 0)
+		(unit 1)
+		(exclude_from_sim no)
+		(in_bom yes)
+		(on_board yes)
+		(dnp no)
+		(fields_autoplaced yes)
+		(property "Reference" "U1"
+			(at 50.4033 38.1 0)
+			(effects
+				(font
+					(size 1.27 1.27)
+				)
+				(justify left)
+			)
+		)
+		(property "Value" "74LS192"
+			(at 50.4033 40.64 0)
+			(effects
+				(font
+					(size 1.27 1.27)
+				)
+				(justify left)
+			)
+		)
+		(property "Footprint" ""
+			(at 48.26 55.88 0)
+			(effects
+				(font
+					(size 1.27 1.27)
+				)
+				(hide yes)
+			)
+		)
+		(property "Datasheet" "http://www.ti.com/lit/ds/symlink/sn74ls193.pdf"
+			(at 48.26 55.88 0)
+			(effects
+				(font
+					(size 1.27 1.27)
+				)
+				(hide yes)
+			)
+		)
+		(property "Description" "Synchronous 4-bit Up/Down (2 clk) counter"
+			(at 48.26 55.88 0)
+			(effects
+				(font
+					(size 1.27 1.27)
+				)
+				(hide yes)
+			)
+		)
+		(pin "6"
+		)
+		(pin "13"
+		)
+		(pin "16"
+		)
+		(pin "7"
+		)
+		(pin "2"
+		)
+		(pin "14"
+		)
+		(pin "3"
+		)
+		(pin "8"
+		)
+		(pin "9"
+		)
+		(pin "11"
+		)
+		(pin "1"
+		)
+		(pin "12"
+		)
+		(pin "5"
+		)
+		(pin "4"
+		)
+		(pin "10"
+		)
+		(pin "15"
+		)
+		(instances
+			(project ""
+				(path "/79d96a8f-9c80-4f83-a25e-7a8fff40baf7/237a212b-f9ce-4ec4-8760-74ac913d696e/4e052793-2ff8-4f97-9964-b86eae475438"
+					(reference "U1")
+					(unit 1)
+				)
+			)
+		)
+	)
 )

Commit message: uodate
Parts:
- removed U1: 74LS192, symbol 74xx:74LS192
- added C7: 0.1uF, symbol Device:C_Small
- added U1: 74LS390, symbol 74xx:74LS390
Connections:
- new net: U1.12 (~{CP1}), U1.13 (Q0)
- new net +5V: C7.1, U1.16 (VCC)
- new net Clock: U1.1 (~{CP0})
- new net GND: C7.2, U1.8 (GND)
- new net Q1S_A: U1.3 (Q0), U1.4 (~{CP1})
- new net Q1S_B: U1.5 (Q1)
- new net Q1S_C: U1.6 (Q2)
- new net Q1S_D: U1.7 (Q3)
Other:
- note added: "Low if no Reset signal"
- note added: "MOD-10 Counter"
- note added: "MOD-6 Counter"
